File: Hardware/PoppyIO/inputs.kicad_sch (KiCad schematic)
At the start: 102 parts

Commit message: hw: io: Updates
Parts:
- J? (x4): value (none) -> WAGO 233-508
Changed lines of the file:
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@@
       (effects (font (size 1.27 1.27)) (justify left))
     )
-    (property "Value" "" (id 1) (at 66.04 60.9599 0)
+    (property "Value" "WAGO 233-508" (id 1) (at 66.04 60.9599 0)
       (effects (font (size 1.27 1.27)) (justify left))
     )
@@
       (effects (font (size 1.27 1.27)) (justify left))
     )
-    (property "Value" "" (id 1) (at 66.04 26.6699 0)
+    (property "Value" "WAGO 233-508" (id 1) (at 66.04 26.6699 0)
       (effects (font (size 1.27 1.27)) (justify left))
     )
@@
       (effects (font (size 1.27 1.27)) (justify left))
     )
-    (property "Value" "" (id 1) (at 66.04 38.0999 0)
+    (property "Value" "WAGO 233-508" (id 1) (at 66.04 38.0999 0)
       (effects (font (size 1.27 1.27)) (justify left))
     )
@@
       (effects (font (size 1.27 1.27)) (justify left))
     )
-    (property "Value" "" (id 1) (at 66.04 49.5299 0)
-      (effects (font (size 1.27 1.27)) (justify left))
-    )
+    (property "Value" "WAGO 233-508" (id 1) (at 66.04 49.5299 0)
+      (effects (font (size 1.27 1.27)) (justify left))
+    )
