File: Hardware/PoppyIO/outputs.kicad_sch (KiCad schematic)
At the start: 8 parts

Commit message: hw: io: Updates
Parts:
- R?: value (none) -> DNP
Changed lines of the file:
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@@
       (effects (font (size 1.27 1.27)) (justify left))
     )
-    (property "Value" "" (id 1) (at 25.4 34.2899 0)
+    (property "Value" "DNP" (id 1) (at 25.4 34.2899 0)
       (effects (font (size 1.27 1.27)) (justify left))
     )
