File: Hardware/PoppyIO/picomcu.kicad_sch (KiCad schematic)
At the start: 1 part

Commit message: hw: io: Updates
Parts:
- added C? (x2): (no value), symbol Device:C_Small
- added D?: (no value), symbol Device:D_Schottky_Small
- added JP?: (no value), symbol Jumper:Jumper_2_Bridged
- added R?: (no value), symbol Device:R_Small
- added SW?: (no value), symbol Switch:SW_Push
Connections:
- net GND: now reaches U?.13 (GND)
- net GND: now also U?.18 (GND), U?.23 (GND), U?.28 (GND), U?.3 (GND), U?.33 (AGND), U?.38 (GND), U?.8 (GND), C?.2, C?.2, SW?.2
- net ~{RESET}: now reaches U?.30 (RUN)
- net ~{RESET}: now also C?.1, R?.2, SW?.1
- net +3V3: now reaches U?.36 (3V3)
- net +3V3: now also R?.1
- net VSYS: now reaches U?.39 (VSYS)
- net VSYS: now also D?.1 (K)
- new net: C?.1, D?.2 (A), JP?.2 (B)
- new net +5V: JP?.1 (A)
- no-connect marks 0 -> 6
Other:
- moved on the sheet: U?
