File: Hardware/PoppyIO/PoppyIO.kicad_pcb (KiCad board)
At the start: 2 copper layers, 102 x 86 mm, 101 parts, among them J1 TC2030-IDC, J10 WAGO 233-508, J11 WAGO 233-508, J12 Conn_02x04_Counter_Clockwise, J2 WAGO 233-508, J3 WAGO 233-508, J4 WAGO 233-508, J5 WAGO 233-508, J6 WAGO 233-508, J7 WAGO 233-508, J8 WAGO 233-508, J9 WAGO 233-508, Q1 FC6946010R, Q2 FC6946010R, Q3 FC6946010R, Q4 FC6946010R, Q5 FC6946010R, Q6 FC6946010R, Q7 FC6946010R, Q8 FC6946010R, SW1 PTS645SH43SMTR92LFS, U1 Pico, U2 PCA9555PW, U3 PCA9555PW, U4 ULQ2003A, U5 ULQ2003A, U6 ULQ2003A

Commit message: hw: io: Updates
Parts:
- added R21: 680k, Resistor_SMD:R_0603_1608Metric_Pad0.98x0.95mm_HandSolder, F.Cu at (119.4, 70.1)
- added R22: 100k, Resistor_SMD:R_0603_1608Metric_Pad0.98x0.95mm_HandSolder, F.Cu at (119.4, 73.6)
- added R23: 680k, Resistor_SMD:R_0603_1608Metric_Pad0.98x0.95mm_HandSolder, F.Cu at (121.9, 70.1)
- added R24: 100k, Resistor_SMD:R_0603_1608Metric_Pad0.98x0.95mm_HandSolder, F.Cu at (121.9, 73.6)
- added R27: 680k, Resistor_SMD:R_0603_1608Metric_Pad0.98x0.95mm_HandSolder, F.Cu at (124.5, 70.1)
- added R28: 100k, Resistor_SMD:R_0603_1608Metric_Pad0.98x0.95mm_HandSolder, F.Cu at (124.5, 73.6)
- added R29: 680k, Resistor_SMD:R_0603_1608Metric_Pad0.98x0.95mm_HandSolder, F.Cu at (127.0, 70.1)
- added R30: 100k, Resistor_SMD:R_0603_1608Metric_Pad0.98x0.95mm_HandSolder, F.Cu at (127.0, 73.6)
- added R33: 680k, Resistor_SMD:R_0603_1608Metric_Pad0.98x0.95mm_HandSolder, F.Cu at (132.4, 70.1)
- added R34: 100k, Resistor_SMD:R_0603_1608Metric_Pad0.98x0.95mm_HandSolder, F.Cu at (132.4, 73.6)
- added R35: 680k, Resistor_SMD:R_0603_1608Metric_Pad0.98x0.95mm_HandSolder, F.Cu at (134.9, 70.1)
- added R36: 100k, Resistor_SMD:R_0603_1608Metric_Pad0.98x0.95mm_HandSolder, F.Cu at (134.9, 73.6)
- added R39: 680k, Resistor_SMD:R_0603_1608Metric_Pad0.98x0.95mm_HandSolder, F.Cu at (137.5, 70.1)
- added R40: 100k, Resistor_SMD:R_0603_1608Metric_Pad0.98x0.95mm_HandSolder, F.Cu at (137.5, 73.6)
- added R41: 680k, Resistor_SMD:R_0603_1608Metric_Pad0.98x0.95mm_HandSolder, F.Cu at (140.0, 70.1)
- added R42: 100k, Resistor_SMD:R_0603_1608Metric_Pad0.98x0.95mm_HandSolder, F.Cu at (140.0, 73.6)
- added R45: 680k, Resistor_SMD:R_0603_1608Metric_Pad0.98x0.95mm_HandSolder, F.Cu at (145.4, 70.1)
- added R46: 100k, Resistor_SMD:R_0603_1608Metric_Pad0.98x0.95mm_HandSolder, F.Cu at (145.4, 73.6)
- added R47: 680k, Resistor_SMD:R_0603_1608Metric_Pad0.98x0.95mm_HandSolder, F.Cu at (147.9, 70.1)
- added R48: 100k, Resistor_SMD:R_0603_1608Metric_Pad0.98x0.95mm_HandSolder, F.Cu at (147.9, 73.6)
- added R51: 680k, Resistor_SMD:R_0603_1608Metric_Pad0.98x0.95mm_HandSolder, F.Cu at (150.5, 70.1)
- added R52: 100k, Resistor_SMD:R_0603_1608Metric_Pad0.98x0.95mm_HandSolder, F.Cu at (150.5, 73.6)
- added R53: 680k, Resistor_SMD:R_0603_1608Metric_Pad0.98x0.95mm_HandSolder, F.Cu at (153.0, 70.1)
- added R54: 100k, Resistor_SMD:R_0603_1608Metric_Pad0.98x0.95mm_HandSolder, F.Cu at (153.0, 73.6)
- moved Q6 3.43 mm to (138.7, 76.7), turned to 0 degrees
- moved Q4 3.28 mm to (125.7, 76.7), turned to 0 degrees
- moved Q5 3.20 mm to (133.7, 76.7), turned to 0 degrees
- moved Q8 3.19 mm to (151.7, 76.7), turned to 0 degrees
- moved Q3 3.19 mm to (120.7, 76.7), turned to 0 degrees
- moved Q7 3.19 mm to (146.7, 76.7), turned to 0 degrees
- moved U2 0.71 mm to (130.0, 94.5)
- moved U3 0.71 mm to (130.0, 105.5)
Routing:
- net GND: track 14.9 -> 86.5 mm, vias 4 -> 14
- net /I14_LOW: track 0.00 -> 48.3 mm, vias 0 -> 2
- net /I15_LOW: track 0.00 -> 46.4 mm, vias 0 -> 2
- net /O00_LOW: track 0.00 -> 44.9 mm
- net /I12_LOW: track 0.00 -> 44.8 mm, vias 0 -> 2
- net /I13_LOW: track 0.00 -> 42.6 mm, vias 0 -> 2
- net /O01_LOW: track 0.00 -> 40.9 mm
- net /I10_LOW: track 0.00 -> 38.0 mm, vias 0 -> 2
- net /I04_LOW: track 0.00 -> 37.1 mm, vias 0 -> 2
- net /O02_LOW: track 0.00 -> 36.8 mm
- net /I11_LOW: track 0.00 -> 35.9 mm, vias 0 -> 2
- net /I08_LOW: track 0.00 -> 35.7 mm, vias 0 -> 2
- net /O15_LOW: track 0.00 -> 35.7 mm
- net /I06_LOW: track 0.00 -> 33.1 mm, vias 0 -> 2
- net /O14_LOW: track 0.00 -> 33.0 mm
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Other:
- board text added: "I00"
- board text added: "I01"
- board text added: "I02"
- board text added: "I03"
- board text added: "I04"
- board text added: "I05"
- board text added: "I06"
- board text added: "I07"
- board text added: "I08"
- board text added: "I09"
- board text added: "I10"
- board text added: "I11"
- board text added: "I12"
- board text added: "I13"
- board text added: "I14"
- board text added: "I15"
- board text added: "O00"
- board text added: "O01"
- board text added: "O02"
- board text added: "O03"
- board text added: "O04"
- board text added: "O05"
- board text added: "O06"
- board text added: "O07"
- board text added: "O08"
- board text added: "O09"
- board text added: "O10"
- board text added: "O11"
- board text added: "O12"
- board text added: "O13"
- board text added: "O14"
- board text added: "O15"

Commit message: hw: io: Update PCB
Parts:
- added C1: 47u, Capacitor_SMD:C_1210_3225Metric, F.Cu at (66.5, 95.0)
- added C2: DNP, Capacitor_SMD:C_0603_1608Metric_Pad1.08x0.95mm_HandSolder, F.Cu at (89.0, 89.0)
- added C3: DNP, Capacitor_SMD:C_0603_1608Metric_Pad1.08x0.95mm_HandSolder, F.Cu at (75.7, 96.2)
- added C4: 100n, Capacitor_SMD:C_0603_1608Metric_Pad1.08x0.95mm_HandSolder, F.Cu at (75.7, 98.7)
- added C5: 100n, Capacitor_SMD:C_0603_1608Metric_Pad1.08x0.95mm_HandSolder, F.Cu at (130.0, 89.5)
- added C6: 100n, Capacitor_SMD:C_0603_1608Metric_Pad1.08x0.95mm_HandSolder, F.Cu at (136.8, 102.5)
- added D1: MBR120, Diode_SMD:D_SMB, F.Cu at (59.5, 95.7)
- added JP1: ~, Connector_PinHeader_2.54mm:PinHeader_1x02_P2.54mm_Vertical, F.Cu at (187.5, 70.7)
- added JP2: SolderJumper_2_Bridged, Jumper:SolderJumper-2_P1.3mm_Bridged_RoundedPad1.0x1.5mm, B.Cu at (130.5, 84.0)
- added JP3: SolderJumper_2_Bridged, Jumper:SolderJumper-2_P1.3mm_Bridged_RoundedPad1.0x1.5mm, B.Cu at (130.5, 86.5)
- added JP4: SolderJumper_2_Bridged, Jumper:SolderJumper-2_P1.3mm_Bridged_RoundedPad1.0x1.5mm, B.Cu at (130.5, 89.0)
- added JP5: SolderJumper_2_Open, Jumper:SolderJumper-2_P1.3mm_Open_RoundedPad1.0x1.5mm, B.Cu at (125.5, 108.0)
- added JP6: SolderJumper_2_Bridged, Jumper:SolderJumper-2_P1.3mm_Bridged_RoundedPad1.0x1.5mm, B.Cu at (125.5, 105.5)
- added JP7: SolderJumper_2_Bridged, Jumper:SolderJumper-2_P1.3mm_Bridged_RoundedPad1.0x1.5mm, B.Cu at (125.5, 103.0)
- added R1: 0R, Resistor_SMD:R_0603_1608Metric_Pad0.98x0.95mm_HandSolder, F.Cu at (89.0, 91.5)
- added R2: 0R, Resistor_SMD:R_0603_1608Metric_Pad0.98x0.95mm_HandSolder, F.Cu at (80.3, 91.5)
- added R3: 10k, Resistor_SMD:R_0603_1608Metric_Pad0.98x0.95mm_HandSolder, F.Cu at (84.3, 95.1)
- added R4: DNP, Resistor_SMD:R_0603_1608Metric_Pad0.98x0.95mm_HandSolder, F.Cu at (167.0, 80.5)
- added R5: 4.7k, Resistor_SMD:R_0603_1608Metric_Pad0.98x0.95mm_HandSolder, F.Cu at (150.2, 101.2)
- added R6: 4.7k, Resistor_SMD:R_0603_1608Metric_Pad0.98x0.95mm_HandSolder, F.Cu at (150.2, 102.8)
- added R7: DNP, Resistor_SMD:R_0603_1608Metric_Pad0.98x0.95mm_HandSolder, F.Cu at (124.5, 90.2)
- added R8: DNP, Resistor_SMD:R_0603_1608Metric_Pad0.98x0.95mm_HandSolder, F.Cu at (125.2, 102.0)
- added TP1: TestPoint, TestPoint:TestPoint_THTPad_D1.0mm_Drill0.5mm, F.Cu at (75.0, 70.2)
- added TP2: TestPoint, TestPoint:TestPoint_THTPad_D1.0mm_Drill0.5mm, F.Cu at (75.5, 74.2)
- moved SW1 38.7 mm to (223.8, 85.2)
- moved J7 24.0 mm to (162.0, 135.0)
- moved U1 17.0 mm to (186.0, 117.0)
Connections:
- U5 pad 1: /O13_LOW -> unconnected-(U5-Pad1)
- U5 pad 15: O12_HIGH -> unconnected-(U5-Pad15)
- U5 pad 16: O13_HIGH -> unconnected-(U5-Pad16)
- U5 pad 2: /O12_LOW -> unconnected-(U5-Pad2)
- U6 pad 13: unconnected-(U6-Pad13) -> O12_HIGH
- U6 pad 14: unconnected-(U6-Pad14) -> O13_HIGH
- U6 pad 3: unconnected-(U6-Pad3) -> /O13_LOW
- U6 pad 4: unconnected-(U6-Pad4) -> /O12_LOW
Routing:
- net +3V3: track 0.00 -> 108.3 mm, vias 0 -> 1
- net +24V: track 15.1 -> 57.5 mm, vias 0 -> 3
- net IO_SCL: track 0.00 -> 36.1 mm, vias 0 -> 2
- net GND: track 86.5 -> 116.7 mm, vias 14 -> 58
- net IO_SDA: track 0.00 -> 29.2 mm, vias 0 -> 2
- net ~{INT_INPUT}: track 0.00 -> 28.8 mm, vias 0 -> 2
- net ~{INT_OUTPUT}: track 0.00 -> 24.4 mm
- net Net-(U2-Pad21): track 0.00 -> 18.9 mm, vias 0 -> 1
- net +5V: track 15.1 -> 0.00 mm
- net Net-(U3-Pad2): track 0.00 -> 9.28 mm, vias 0 -> 1
- net Net-(U3-Pad21): track 0.00 -> 8.77 mm, vias 0 -> 1
- net O15_HIGH: track 5.00 -> 13.2 mm
- net O14_HIGH: track 5.00 -> 12.0 mm
- net Net-(U2-Pad2): track 0.00 -> 6.98 mm, vias 0 -> 1
- net /O15_LOW: track 35.7 -> 42.5 mm
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- added copper zone on B.Cu, net +24V
- added copper zone on F.Cu, net +24V
- added copper zone on B.Cu, net +5V
- added copper zone on F.Cu, net +5V
- added copper zone on B.Cu, net GND
- added copper zone on F.Cu, net GND

Commit message: hw: io: PCB Updates
Parts:
- moved D1 132.5 mm to (191.5, 84.0), turned to 90 degrees
- moved C1 108.7 mm to (170.2, 127.5), turned to 90 degrees
- moved TP1 101.3 mm to (168.5, 109.2)
- moved TP2 98.6 mm to (168.5, 107.0)
- moved C4 94.7 mm to (168.0, 119.8), turned to 180 degrees
- moved C3 94.0 mm to (169.5, 90.5), turned to 180 degrees
- moved R2 89.2 mm to (169.5, 92.0), turned to 180 degrees
- moved R3 87.7 mm to (168.0, 121.2)
- moved C2 80.7 mm to (169.5, 95.0), turned to 180 degrees
- moved R1 80.5 mm to (169.5, 93.5), turned to 180 degrees
- moved SW1 66.5 mm to (164.5, 115.5), turned to 180 degrees
- moved J12 25.8 mm to (161.5, 67.0)
- moved R4 14.9 mm to (163.4, 95.0)
- moved J1 14.9 mm to (165.5, 100.0)
- moved R7 12.0 mm to (122.0, 102.0), turned to 90 degrees
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Connections:
- C1 pad 1: Net-(C1-Pad1) -> /VSYS
- D1 pad 2: Net-(C1-Pad1) -> Net-(JP1-Pad2)
- JP1 pad 2: Net-(C1-Pad1) -> Net-(JP1-Pad2)
Routing:
- net +3V3: track 108.3 -> 229.8 mm, vias 1 -> 6
- net /VSYS: track 0.00 -> 73.1 mm
- net IO_SDA: track 29.2 -> 86.0 mm
- net IO_SCL: track 36.1 -> 85.5 mm
- net /SWCLK: track 3.53 -> 51.9 mm, vias 0 -> 2
- net /~{RESET}: track 4.03 -> 41.8 mm, vias 0 -> 2
- net /SWDIO: track 2.44 -> 38.2 mm, vias 0 -> 2
- net GND: track 116.7 -> 152.0 mm, vias 58 -> 59
- net ~{INT_INPUT}: track 28.8 -> 62.3 mm
- net ~{INT_OUTPUT}: track 24.4 -> 56.0 mm, vias 0 -> 2
- net +5V: track 0.00 -> 11.1 mm
- net Net-(C2-Pad1): track 0.00 -> 9.01 mm
- net Net-(C3-Pad1): track 0.00 -> 8.58 mm
- net Net-(JP1-Pad2): track 0.00 -> 7.45 mm
- net Net-(U3-Pad2): track 9.28 -> 10.7 mm
Other:
- board text added: "+24"
- board text added: "+5V"
- board text added: "G"
- board text added: "GND"

Commit message: hw: io: More updates
Parts:
- removed R4: DNP, Resistor_SMD:R_0603_1608Metric_Pad0.98x0.95mm_HandSolder
- added JP8: SolderJumper_2_Bridged, Jumper:SolderJumper-2_P1.3mm_Bridged2Bar_RoundedPad1.0x1.5mm, F.Cu at (162.2, 122.5)
- J10, J11, J2, J3, J4, J5, J6, J7, J8, J9: value WAGO 233-508 -> WAGO 233-504
- J12: value Conn_02x04_Counter_Clockwise -> ~
- moved J12 13.1 mm to (162.5, 80.0), turned to 90 degrees
- moved C4 1.50 mm to (168.0, 121.2)
- moved R3 1.50 mm to (168.0, 119.8)
Connections:
- J1 pad 6: Net-(J1-Pad6) -> unconnected-(J1-Pad6)
- J12 pad 2: ~{INT_INPUT} -> +3V3
- J12 pad 3: ~{INT_OUTPUT} -> ~{INT_INPUT}
- J12 pad 4: GND -> IO_SCL
- J12 pad 5: GND -> ~{INT_OUTPUT}
- J12 pad 7: IO_SCL -> GND
- J12 pad 8: +3V3 -> GND
- J2 pad 1: +5V -> GND
- J2 pad 2: +5V -> GND
- J2 pad 3: GND -> +5V
- J2 pad 4: GND -> +5V
- U1 pad 36: +3V3 -> Net-(U1-Pad36)
Routing:
- net +5V: track 11.1 -> 44.2 mm, vias 0 -> 2
- net IO_SDA: track 86.0 -> 114.7 mm, vias 2 -> 3
- net IO_SCL: track 85.5 -> 111.5 mm, vias 2 -> 3
- net Net-(U1-Pad36): track 0.00 -> 21.5 mm
- net ~{INT_OUTPUT}: track 56.0 -> 70.0 mm, vias 2 -> 3
- net ~{INT_INPUT}: track 62.3 -> 74.3 mm, vias 2 -> 3
- net +3V3: track 229.8 -> 235.0 mm, vias 6 -> 7
- net GND: track 152.0 -> 152.2 mm, vias 59 -> 111
