File: Hardware/PoppyIO/PoppyIO.kicad_sch (KiCad schematic)
At the start: 250 parts, among them J1 WAGO 233-504, J10 Phoenix MPT 0,5/ 4-2,54, J11 TC2030-IDC, J12 Conn_02x06_Odd_Even, J2 WAGO 233-504, J3 WAGO 233-504, J4 WAGO 233-504, J5 WAGO 233-504, J6 WAGO 233-504, J7 WAGO 233-504, J8 WAGO 233-504, J9 Phoenix MPT 0,5/ 4-2,54, SW1 PTS645SH43SMTR92LFS, U1 Pico, U10 74HC14, U11 74HC14, U12 74HC14, U2 PCA9538PW, U3 PCA9538PW, U4 PCA9538PW, U5 PCA9538PW, U6 ULN2003AD, U7 ULN2003AD, U8 ULN2003AD, U9 74HC14

Commit message: hw: io: Final touches and prepare revision A
Parts:
- C32: value (none) -> 10u; footprint (none) -> Capacitor_SMD:C_1210_3225Metric
- SYM1: value (none) -> SYM_Rahix; footprint (none) -> PoppyLogicController:SYM_Rahix
- U13: value (none) -> LM78xx; footprint (none) -> PoppyLogicController:TO-220-3_Vertical_Clearance
Changed lines of the file:
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@@
   (title_block
     (title "Poppy Logic Controller - IO Board")
-    (date "2022-04-01")
-    (rev "Unreleased")
+    (date "2022-04-24")
+    (rev "A")
   )
   (junction (at 251.46 255.27) (diameter 0) (color 0 0 0 0)
@@
       (effects (font (size 1.27 1.27)) hide)
     )
-    (property "Value" "" (id 1) (at 378.46 46.99 0))
+    (property "Value" "+24V" (id 1) (at 378.46 46.99 0))
     (property "Footprint" "" (id 2) (at 378.46 52.07 0)
       (effects (font (size 1.27 1.27)) hide)
@@
     (in_bom yes) (on_board yes) (fields_autoplaced)
     (property "Reference" "U13" (id 0) (at 387.35 43.18 0))
-    (property "Value" "" (id 1) (at 387.35 45.72 0))
-    (property "Footprint" "" (id 2) (at 387.35 47.625 0)
+    (property "Value" "LM78xx" (id 1) (at 387.35 45.72 0))
+    (property "Footprint" "PoppyLogicController:TO-220-3_Vertical_Clearance" (id 2) (at 387.35 47.625 0)
       (effects (font (size 1.27 1.27) italic) hide)
     )
@@
       (effects (font (size 1.27 1.27)) hide)
     )
-    (property "Value" "" (id 1) (at 394.8684 231.6226 0)
+    (property "Value" "SYM_Rahix" (id 1) (at 394.8684 231.6226 0)
       (effects (font (size 1.27 1.27)) hide)
     )
-    (property "Footprint" "" (id 2) (at 387.35 238.76 0)
+    (property "Footprint" "PoppyLogicController:SYM_Rahix" (id 2) (at 387.35 238.76 0)
       (effects (font (size 1.27 1.27)) hide)
     )
@@
       (effects (font (size 1.27 1.27)) (justify right))
     )
-    (property "Value" "" (id 1) (at 375.92 57.1562 0)
+    (property "Value" "10u" (id 1) (at 375.92 57.1562 0)
       (effects (font (size 1.27 1.27)) (justify right))
     )
-    (property "Footprint" "" (id 2) (at 378.46 57.15 0)
+    (property "Footprint" "Capacitor_SMD:C_1210_3225Metric" (id 2) (at 378.46 57.15 0)
       (effects (font (size 1.27 1.27)) hide)
     )

Commit message: hw: io: Switch to 14-pin IDC
Parts:
- J12: value Conn_02x06_Odd_Even -> (none); footprint Connector_IDC:IDC-Header_2x06_P2.54mm_Vertical -> (none); symbol Connector_Generic:Conn_02x06_Odd_Even -> Connector_Generic:Conn_02x07_Odd_Even
Connections:
- net +3V3: now also J12.4 (Pin_4)
- net +5V: now also J12.3 (Pin_3)
- net GND: now also J12.13 (Pin_13), J12.14 (Pin_14); no longer J12.10 (Pin_10), J12.11 (Pin_11)
- net IO_INT0: now also J12.7 (Pin_7); no longer J12.5 (Pin_5)
- net IO_INT1: now also J12.9 (Pin_9); no longer J12.7 (Pin_7)
- net IO_SCL: now also J12.6 (Pin_6); no longer J12.4 (Pin_4)
- net IO_SDA: now also J12.8 (Pin_8); no longer J12.6 (Pin_6)
- net PICO_RX: now also J12.11 (Pin_11); no longer J12.9 (Pin_9)
- net PICO_TX: now also J12.10 (Pin_10); no longer J12.8 (Pin_8)
- net at R73.2: now also J12.5 (Pin_5); no longer J12.3 (Pin_3)
Other:
- moved on the sheet: R73

Commit message: hw: io: Prepare revision B
Other:
- company: (none) -> Rahix
Changed lines of the file:
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@@
   (title_block
     (title "Poppy Logic Controller - IO Board")
-    (date "2022-04-24")
-    (rev "A")
+    (date "2022-04-25")
+    (rev "B")
+    (company "Rahix")
   )
   (junction (at 251.46 255.27) (diameter 0) (color 0 0 0 0)

Commit message: hw: io: Fix wrong DI resistors
Copy-paste error - the calculations projected an 820Ω resistor but I
accidentally used 680Ω instead.  This still works but has different
limiting values...
Parts:
- J12: value (none) -> Conn_02x07_Odd_Even; footprint (none) -> Connector_IDC:IDC-Header_2x07_P2.54mm_Vertical
- R10, R11, R12, R21, R22, R23, R24, R33, R34, R35, R36, R45, R46, R47, R48, R9: value 680 250mW -> 820 250mW
Changed lines of the file:
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@@
   (title_block
     (title "Poppy Logic Controller - IO Board")
-    (date "2022-04-25")
-    (rev "B")
+    (date "2022-06-26")
+    (rev "C")
     (company "Rahix")
   )
@@
     (in_bom yes) (on_board yes) (fields_autoplaced)
     (property "Reference" "J12" (id 0) (at 330.2 17.78 0))
-    (property "Value" "" (id 1) (at 330.2 20.32 0)
+    (property "Value" "Conn_02x07_Odd_Even" (id 1) (at 330.2 20.32 0)
       (effects (font (size 1.27 1.27)) hide)
     )
-    (property "Footprint" "" (id 2) (at 328.93 29.21 0)
+    (property "Footprint" "Connector_IDC:IDC-Header_2x07_P2.54mm_Vertical" (id 2) (at 328.93 29.21 0)
       (effects (font (size 1.27 1.27)) hide)
     )
@@
       (effects (font (size 1.27 1.27)) (justify right))
     )
-    (property "Value" "680 250mW" (id 1) (at 130.81 190.4999 0)
+    (property "Value" "820 250mW" (id 1) (at 130.81 190.4999 0)
       (effects (font (size 1.27 1.27)) (justify right))
     )
@@
       (effects (font (size 1.27 1.27)) (justify right))
     )
-    (property "Value" "680 250mW" (id 1) (at 257.81 214.6299 0)
+    (property "Value" "820 250mW" (id 1) (at 257.81 214.6299 0)
       (effects (font (size 1.27 1.27)) (justify right))
     )
@@
       (effects (font (size 1.27 1.27)) (justify right))
     )
-    (property "Value" "680 250mW" (id 1) (at 194.31 238.7599 0)
+    (property "Value" "820 250mW" (id 1) (at 194.31 238.7599 0)
       (effects (font (size 1.27 1.27)) (justify right))
     )
@@
       (effects (font (size 1.27 1.27)) (justify right))
     )
-    (property "Value" "680 250mW" (id 1) (at 67.31 190.4999 0)
+    (property "Value" "820 250mW" (id 1) (at 67.31 190.4999 0)
       (effects (font (size 1.27 1.27)) (justify right))
     )
@@
       (effects (font (size 1.27 1.27)) (justify right))
     )
-    (property "Value" "680 250mW" (id 1) (at 194.31 190.4999 0)
+    (property "Value" "820 250mW" (id 1) (at 194.31 190.4999 0)
       (effects (font (size 1.27 1.27)) (justify right))
     )
@@
       (effects (font (size 1.27 1.27)) (justify right))
     )
-    (property "Value" "680 250mW" (id 1) (at 67.31 238.7599 0)
+    (property "Value" "820 250mW" (id 1) (at 67.31 238.7599 0)
       (effects (font (size 1.27 1.27)) (justify right))
     )
@@
       (effects (font (size 1.27 1.27)) (justify right))
     )
-    (property "Value" "680 250mW" (id 1) (at 194.31 262.8899 0)
+    (property "Value" "820 250mW" (id 1) (at 194.31 262.8899 0)
       (effects (font (size 1.27 1.27)) (justify right))
     )
@@
       (effects (font (size 1.27 1.27)) (justify right))
     )
-    (property "Value" "680 250mW" (id 1) (at 194.31 214.6299 0)
+    (property "Value" "820 250mW" (id 1) (at 194.31 214.6299 0)
       (effects (font (size 1.27 1.27)) (justify right))
     )
@@
       (effects (font (size 1.27 1.27)) (justify right))
     )
-    (property "Value" "680 250mW" (id 1) (at 130.81 262.8899 0)
+    (property "Value" "820 250mW" (id 1) (at 130.81 262.8899 0)
       (effects (font (size 1.27 1.27)) (justify right))
     )
@@
       (effects (font (size 1.27 1.27)) (justify right))
     )
-    (property "Value" "680 250mW" (id 1) (at 257.81 262.8899 0)
+    (property "Value" "820 250mW" (id 1) (at 257.81 262.8899 0)
       (effects (font (size 1.27 1.27)) (justify right))
     )
@@
       (effects (font (size 1.27 1.27)) (justify right))
     )
-    (property "Value" "680 250mW" (id 1) (at 257.81 238.7599 0)
+    (property "Value" "820 250mW" (id 1) (at 257.81 238.7599 0)
       (effects (font (size 1.27 1.27)) (justify right))
     )
@@
       (effects (font (size 1.27 1.27)) (justify right))
     )
-    (property "Value" "680 250mW" (id 1) (at 67.31 262.8899 0)
+    (property "Value" "820 250mW" (id 1) (at 67.31 262.8899 0)
       (effects (font (size 1.27 1.27)) (justify right))
     )
@@
       (effects (font (size 1.27 1.27)) (justify right))
     )
-    (property "Value" "680 250mW" (id 1) (at 130.81 214.6299 0)
+    (property "Value" "820 250mW" (id 1) (at 130.81 214.6299 0)
       (effects (font (size 1.27 1.27)) (justify right))
     )
@@
       (effects (font (size 1.27 1.27)) (justify right))
     )
-    (property "Value" "680 250mW" (id 1) (at 67.31 214.6299 0)
+    (property "Value" "820 250mW" (id 1) (at 67.31 214.6299 0)
       (effects (font (size 1.27 1.27)) (justify right))
     )
@@
       (effects (font (size 1.27 1.27)) (justify right))
     )
-    (property "Value" "680 250mW" (id 1) (at 130.81 238.7599 0)
+    (property "Value" "820 250mW" (id 1) (at 130.81 238.7599 0)
       (effects (font (size 1.27 1.27)) (justify right))
     )
@@
       (effects (font (size 1.27 1.27)) (justify right))
     )
-    (property "Value" "680 250mW" (id 1) (at 257.81 190.4999 0)
+    (property "Value" "820 250mW" (id 1) (at 257.81 190.4999 0)
       (effects (font (size 1.27 1.27)) (justify right))
     )
@@
     )
     (path "/56dc8e49-e8ba-4a80-ae70-4c19274985ce"
-      (reference "R9") (unit 1) (value "680 250mW") (footprint "Resistor_SMD:R_1206_3216Metric")
+      (reference "R9") (unit 1) (value "820 250mW") (footprint "Resistor_SMD:R_1206_3216Metric")
     )
     (path "/e5391d8e-da72-42a1-90ac-b47abf0b024a"
-      (reference "R10") (unit 1) (value "680 250mW") (footprint "Resistor_SMD:R_1206_3216Metric")
+      (reference "R10") (unit 1) (value "820 250mW") (footprint "Resistor_SMD:R_1206_3216Metric")
     )
     (path "/72696289-14d4-4dd3-84f2-08cf4925c569"
-      (reference "R11") (unit 1) (value "680 250mW") (footprint "Resistor_SMD:R_1206_3216Metric")
+      (reference "R11") (unit 1) (value "820 250mW") (footprint "Resistor_SMD:R_1206_3216Metric")
     )
     (path "/c7537f41-8140-4148-affd-730249022f3d"
-      (reference "R12") (unit 1) (value "680 250mW") (footprint "Resistor_SMD:R_1206_3216Metric")
+      (reference "R12") (unit 1) (value "820 250mW") (footprint "Resistor_SMD:R_1206_3216Metric")
     )
     (path "/3916062a-93a1-4262-b4bc-59b8bd7bf167"
@@
     )
     (path "/02872268-7d42-47a7-b6a6-e8c7e3ebbb3b"
-      (reference "R21") (unit 1) (value "680 250mW") (footprint "Resistor_SMD:R_1206_3216Metric")
+      (reference "R21") (unit 1) (value "820 250mW") (footprint "Resistor_SMD:R_1206_3216Metric")
     )
     (path "/cc0e6a6d-b74c-4a7a-91ba-c5442ef44c19"
-      (reference "R22") (unit 1) (value "680 250mW") (footprint "Resistor_SMD:R_1206_3216Metric")
+      (reference "R22") (unit 1) (value "820 250mW") (footprint "Resistor_SMD:R_1206_3216Metric")
     )
     (path "/f2a3e53a-5dd3-41c8-a51c-580e4033b9c1"
-      (reference "R23") (unit 1) (value "680 250mW") (footprint "Resistor_SMD:R_1206_3216Metric")
+      (reference "R23") (unit 1) (value "820 250mW") (footprint "Resistor_SMD:R_1206_3216Metric")
     )
     (path "/86b51b27-9969-4258-9bb3-f3653d4ea4d5"
-      (reference "R24") (unit 1) (value "680 250mW") (footprint "Resistor_SMD:R_1206_3216Metric")
+      (reference "R24") (unit 1) (value "820 250mW") (footprint "Resistor_SMD:R_1206_3216Metric")
     )
     (path "/d4565a4b-3d2d-40c3-981b-61e8ec468f40"
@@
     )
     (path "/6a366be5-8068-4186-a770-7cbf78c6b522"
-      (reference "R33") (unit 1) (value "680 250mW") (footprint "Resistor_SMD:R_1206_3216Metric")
+      (reference "R33") (unit 1) (value "820 250mW") (footprint "Resistor_SMD:R_1206_3216Metric")
     )
     (path "/7db7eeba-4878-49f0-9a33-7d0982cbf8c1"
-      (reference "R34") (unit 1) (value "680 250mW") (footprint "Resistor_SMD:R_1206_3216Metric")
+      (reference "R34") (unit 1) (value "820 250mW") (footprint "Resistor_SMD:R_1206_3216Metric")
     )
     (path "/3e35923b-0e46-4736-8682-abd41e72ba05"
-      (reference "R35") (unit 1) (value "680 250mW") (footprint "Resistor_SMD:R_1206_3216Metric")
+      (reference "R35") (unit 1) (value "820 250mW") (footprint "Resistor_SMD:R_1206_3216Metric")
     )
     (path "/7c0bf56b-59f6-4cd8-96a2-5736cbc9dda0"
-      (reference "R36") (unit 1) (value "680 250mW") (footprint "Resistor_SMD:R_1206_3216Metric")
+      (reference "R36") (unit 1) (value "820 250mW") (footprint "Resistor_SMD:R_1206_3216Metric")
     )
     (path "/83c17841-f60c-4f80-b180-167d41e6c9c6"
@@
     )
     (path "/fdafd3b5-27b1-44a4-bac8-f920a748c758"
-      (reference "R45") (unit 1) (value "680 250mW") (footprint "Resistor_SMD:R_1206_3216Metric")
+      (reference "R45") (unit 1) (value "820 250mW") (footprint "Resistor_SMD:R_1206_3216Metric")
     )
     (path "/2dcbe0a9-3866-40b1-9b6d-e1a84e1d4192"
-      (reference "R46") (unit 1) (value "680 250mW") (footprint "Resistor_SMD:R_1206_3216Metric")
+      (reference "R46") (unit 1) (value "820 250mW") (footprint "Resistor_SMD:R_1206_3216Metric")
     )
     (path "/c6ac22ad-0acc-4e6d-9ad9-ec112ba11608"
-      (reference "R47") (unit 1) (value "680 250mW") (footprint "Resistor_SMD:R_1206_3216Metric")
+      (reference "R47") (unit 1) (value "820 250mW") (footprint "Resistor_SMD:R_1206_3216Metric")
     )
     (path "/86f508dd-095e-44fa-ab47-717e7304e37a"
-      (reference "R48") (unit 1) (value "680 250mW") (footprint "Resistor_SMD:R_1206_3216Metric")
+      (reference "R48") (unit 1) (value "820 250mW") (footprint "Resistor_SMD:R_1206_3216Metric")
     )
     (path "/941aa68c-250b-4bb0-935f-fde426fb4f86"

Commit message: hw: io: Schematic updates
- Drop DNP config from LM78xx regulator and capacitors.
- Removed screw-terminal J9 for external 5V supply.
- Switched +24VDC screw-terminal to 2-pin variant.
- Documented J2 meaning.
Parts:
- removed J9: Phoenix MPT 0,5/ 4-2,54, TerminalBlock_Phoenix:TerminalBlock_Phoenix_MPT-0,5-4-2.54_1x04_P2.54mm_Horizontal, symbol Connector:Screw_Terminal_01x04
- C32, C33, U13: Config DNP -> (none)
- J10: value Phoenix MPT 0,5/ 4-2,54 -> Screw_Terminal_01x02; symbol Connector:Screw_Terminal_01x04 -> Connector:Screw_Terminal_01x02
Connections:
- net +24V: no longer J10.2 (Pin_2)
- net GND: now also J10.2 (Pin_2); no longer J10.3 (Pin_3), J10.4 (Pin_4)
- net +3V3 renamed +3.3V
Other:
- note added: "JP2 should be removed when +3.3V is supplied from the board-to-board connector."
- note added: "Populate C30 or C31 when the 3.3V supply is too unstable."
- note added: "U13 is a LM78xx compatible DC/DC step-down converter (fixed 5V out)."
- note removed: "Populate C30/C31 when the 3.3V supply is too unstable."
- note removed: "U13 is an optional LM78xx compatible DC/DC step-down converter (fixed 5V out). This enables a single 24V supply."
- moved on the sheet: J1, J12, J2, J3, J4, J5, J6, J7, J8, JP2, R73

Commit message: hw: io: PCB cleanup and update J10 footprint
Choose an appropriate screw-terminal for J10 which has 2 pins and 5.08mm
pitch.
Parts:
- J10: value Screw_Terminal_01x02 -> MKDS-1,5-2-5.08; footprint TerminalBlock_Phoenix:TerminalBlock_Phoenix_MPT-0,5-4-2.54_1x04_P2.54mm_Horizontal -> TerminalBlock_Phoenix:TerminalBlock_Phoenix_MKDS-1,5-2-5.08_1x02_P5.08mm_Horizontal
- SW1: value PTS645SH43SMTR92LFS -> PTS645
Changed lines of the file:
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@@
       (effects (font (size 1.27 1.27)) (justify left))
     )
-    (property "Value" "Screw_Terminal_01x02" (id 1) (at 78.74 25.3999 0)
+    (property "Value" "MKDS-1,5-2-5.08" (id 1) (at 78.74 25.3999 0)
       (effects (font (size 1.27 1.27)) (justify left))
     )
-    (property "Footprint" "TerminalBlock_Phoenix:TerminalBlock_Phoenix_MPT-0,5-4-2.54_1x04_P2.54mm_Horizontal" (id 2) (at 76.2 22.86 0)
+    (property "Footprint" "TerminalBlock_Phoenix:TerminalBlock_Phoenix_MKDS-1,5-2-5.08_1x02_P5.08mm_Horizontal" (id 2) (at 76.2 22.86 0)
       (effects (font (size 1.27 1.27)) hide)
     )
@@
     (in_bom yes) (on_board yes) (fields_autoplaced)
     (property "Reference" "SW1" (id 0) (at 392.43 157.48 0))
-    (property "Value" "PTS645SH43SMTR92LFS" (id 1) (at 392.43 160.02 0))
+    (property "Value" "PTS645" (id 1) (at 392.43 160.02 0))
     (property "Footprint" "Button_Switch_SMD:SW_SPST_PTS645" (id 2) (at 392.43 160.02 0)
       (effects (font (size 1.27 1.27)) hide)
@@
     )
     (path "/ac89226c-b873-4964-b60c-6cd96dcd0ab9"
-      (reference "J10") (unit 1) (value "Screw_Terminal_01x02") (footprint "TerminalBlock_Phoenix:TerminalBlock_Phoenix_MPT-0,5-4-2.54_1x04_P2.54mm_Horizontal")
+      (reference "J10") (unit 1) (value "MKDS-1,5-2-5.08") (footprint "TerminalBlock_Phoenix:TerminalBlock_Phoenix_MKDS-1,5-2-5.08_1x02_P5.08mm_Horizontal")
     )
     (path "/3e4be841-f567-4772-9110-1e60f784b0c4"
@@
     )
     (path "/f8c96be1-70b9-4023-b323-701f7eafdbb2"
-      (reference "SW1") (unit 1) (value "PTS645SH43SMTR92LFS") (footprint "Button_Switch_SMD:SW_SPST_PTS645")
+      (reference "SW1") (unit 1) (value "PTS645") (footprint "Button_Switch_SMD:SW_SPST_PTS645")
     )
     (path "/7101c69b-dd19-4bf1-bb0a-108aa3dc9beb"

Commit message: hw: io: Add Reichelt SKUs for all applicable parts
Parts:
- C1, C32, C33: Reichelt SKU (none) -> KEM X5R1210 10U
- C24, C25, C26, C28, C29, C4, C5, C6, C7: Reichelt SKU (none) -> X7R-G0603 100N
- D1: Reichelt SKU (none) -> SKL 14 DIO
- J1, J2, J3, J4, J5, J6, J7, J8: Reichelt SKU (none) -> DG240 2,54-4
- J10: Reichelt SKU (none) -> AKL 101-02
- J12: Config (none) -> DNP; Reichelt SKU (none) -> WSL 14G
- JP1, JP2: Reichelt SKU (none) -> MPE 087-1-002
- R1, R2, R73: Reichelt SKU (none) -> SMD-0603 0
- R13, R14, R15, R16, R25, R26, R27, R28, R37, R38, R39, R40, R49, R50, R51, R52, R53, R54, R55, R56, R57, R58, R59, R60, R61, R62, R63, R64, R65, R66, R67, R68: Reichelt SKU (none) -> SMD-0603 1,0K
- R3, R4, R70, R74, R75, R76, R77, R78, R79, R80, R81, R82, R83, R84, R85, R86, R87, R88, R89: Reichelt SKU (none) -> SMD-0603 10K
- R71, R72: Reichelt SKU (none) -> SMD-0603 4,7K
- U10, U11, U12, U9: Reichelt SKU (none) -> 74VHC 14 D
- U13: Reichelt SKU (none) -> LMO78_05-0.5
- U2, U3, U4, U5: Reichelt SKU (none) -> PCA9538PW
- U6, U7, U8: Reichelt SKU ULN 2003 AD -> ULN 2003 AD SMD
